File: kicad/can_controller.sch (KiCad schematic (older format))
At the start: 41 parts, among them J1 OBD-II Connector, J2 Header for SIM800L, J3 Programming conn, SW1 SW_Push_Dual, U1 AP63205WU-7-2020-02-12_13-05-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, U2 STM32F105RCTx, U3 LMR16006YQ, U4 SN65HVD232, U5 SN65HVD232, Y1 8Mhz

Commit message: Finalize schema. Add and assign footprints. Start PCB layout. It's a mess...
Parts:
- removed C14: 2.2uF, symbol Device:C_Small
- removed C16: 0.1uF, symbol Device:C_Small
- removed C18: 10uF, symbol Device:C_Small
- removed C3: 100nF, symbol Device:C_Small
- removed C4, C6: 22uF, symbol Device:C_Small
- removed D4: MBR120ESFT1G1, symbol Device:D_Schottky_Small
- removed L1: 4.7uH, symbol Device:L_Small
- removed L2: 6.8uH, symbol Device:L_Small
- removed U1: AP63205WU-7-2020-02-12_13-05-37, SOIC_05WU-7, symbol can_controller-rescue:AP63205WU-7-2020-02-12_13-05-37
- removed U3: LMR16006YQ, Package_TO_SOT_SMD:SOT-23-6, symbol Regulator_Switching:LMR16006YQ
- added C13: 4.7uF, Capacitor_SMD:C_1206_3216Metric_Pad1.42x1.75mm_HandSolder, symbol can_controller-rescue:C_Small-Device
- added C14, C2: 100nF, Capacitor_SMD:C_1206_3216Metric_Pad1.42x1.75mm_HandSolder, symbol can_controller-rescue:C_Small-Device
- added C17, C4: 10uF, Capacitor_SMD:C_1206_3216Metric_Pad1.42x1.75mm_HandSolder, symbol can_controller-rescue:C_Small-Device
- added D1, D4: MBR120ESFT1G1, Diode_SMD:D_SOD-123F, symbol can_controller-rescue:D_Schottky_Small-Device
- added L1, L2: 22uH, Resistor_SMD:R_1206_3216Metric_Pad1.42x1.75mm_HandSolder, symbol can_controller-rescue:L_Small-Device
- added R1, R5: 5MR, Resistor_SMD:R_1206_3216Metric_Pad1.42x1.75mm_HandSolder, symbol can_controller-rescue:R_Small-Device
- added R2, R7: 49.9kR, Resistor_SMD:R_1206_3216Metric_Pad1.42x1.75mm_HandSolder, symbol can_controller-rescue:R_Small-Device
- added R3: 9.53kR, Resistor_SMD:R_1206_3216Metric_Pad1.42x1.75mm_HandSolder, symbol can_controller-rescue:R_Small-Device
- added R8: 15.8kR, Resistor_SMD:R_1206_3216Metric_Pad1.42x1.75mm_HandSolder, symbol can_controller-rescue:R_Small-Device
- added U1, U3: AOZ1282CI, Package_SO:SO-6L_10x3.84mm_P1.27mm, symbol can_controller-rescue:AOZ1282CI
- BT1: footprint (none) -> Battery_holder:BU2032SM-JJ-GTR; symbol Device:Battery_Cell -> can_controller-rescue:Battery_Cell-Device
- C1: value 10uF -> 4.7uF; footprint (none) -> Capacitor_SMD:C_1206_3216Metric_Pad1.42x1.75mm_HandSolder; symbol Device:C_Small -> can_controller-rescue:C_Small-Device
- C10: renamed from C11; footprint (none) -> Capacitor_SMD:C_1206_3216Metric_Pad1.42x1.75mm_HandSolder; symbol Device:C_Small -> can_controller-rescue:C_Small-Device
- C11: renamed from C12; footprint (none) -> Capacitor_SMD:C_1206_3216Metric_Pad1.42x1.75mm_HandSolder; symbol Device:C_Small -> can_controller-rescue:C_Small-Device
- C12: renamed from C13; footprint (none) -> Capacitor_SMD:C_1206_3216Metric_Pad1.42x1.75mm_HandSolder; symbol Device:C_Small -> can_controller-rescue:C_Small-Device
- C15, C5: footprint (none) -> Capacitor_SMD:C_1206_3216Metric_Pad1.42x1.75mm_HandSolder; symbol Device:C_Small -> can_controller-rescue:C_Small-Device
- C16: renamed from C17; footprint (none) -> Capacitor_SMD:C_1206_3216Metric_Pad1.42x1.75mm_HandSolder; symbol Device:C_Small -> can_controller-rescue:C_Small-Device
- C3: renamed from C2; footprint (none) -> Capacitor_SMD:C_1206_3216Metric_Pad1.42x1.75mm_HandSolder; symbol Device:C_Small -> can_controller-rescue:C_Small-Device
- C6: renamed from C7; footprint (none) -> Capacitor_SMD:C_1206_3216Metric_Pad1.42x1.75mm_HandSolder; symbol Device:C_Small -> can_controller-rescue:C_Small-Device
- C7: renamed from C8; footprint (none) -> Capacitor_SMD:C_1206_3216Metric_Pad1.42x1.75mm_HandSolder; symbol Device:C_Small -> can_controller-rescue:C_Small-Device
- C8: renamed from C9; footprint (none) -> Capacitor_SMD:C_1206_3216Metric_Pad1.42x1.75mm_HandSolder; symbol Device:C_Small -> can_controller-rescue:C_Small-Device
- C9: renamed from C10; footprint (none) -> Capacitor_SMD:C_1206_3216Metric_Pad1.42x1.75mm_HandSolder; symbol Device:C_Small -> can_controller-rescue:C_Small-Device
- D2: renamed from D1; footprint (none) -> LED_SMD:LED_1206_3216Metric_Pad1.42x1.75mm_HandSolder; symbol Device:LED -> can_controller-rescue:LED-Device
- D3: footprint (none) -> RGB_LED:HV-5RGB60
- F1: footprint 0603 -> Fuse:Fuse_0603_1608Metric_Pad1.05x0.95mm_HandSolder; symbol Device:Fuse -> can_controller-rescue:Fuse-Device
- J1: footprint (none) -> kicad:OBDII; symbol Connector_Generic:Conn_02x08_Top_Bottom -> can_controller-rescue:Conn_02x08_Top_Bottom-Connector_Generic
- J2: footprint (none) -> Connector_PinHeader_2.00mm:PinHeader_1x07_P2.00mm_Vertical; symbol Connector:Conn_01x07_Female -> can_controller-rescue:Conn_01x07_Female-Connector
- J3: footprint (none) -> Connector_PinHeader_2.00mm:PinHeader_1x04_P2.00mm_Vertical; symbol Connector:Conn_01x04_Male -> can_controller-rescue:Conn_01x04_Male-Connector
- JP1, JP2: footprint (none) -> Connector_PinHeader_2.00mm:PinHeader_1x02_P2.00mm_Vertical; symbol Device:Jumper_NO_Small -> can_controller-rescue:Jumper_NO_Small-Device
- R10: renamed from R4; footprint (none) -> Resistor_SMD:R_1206_3216Metric_Pad1.42x1.75mm_HandSolder; symbol Device:R_Small -> can_controller-rescue:R_Small-Device
- R4: renamed from R1; footprint (none) -> Resistor_SMD:R_1206_3216Metric_Pad1.42x1.75mm_HandSolder; symbol Device:R_Small -> can_controller-rescue:R_Small-Device
- R6: renamed from R2; footprint (none) -> Resistor_SMD:R_1206_3216Metric_Pad1.42x1.75mm_HandSolder; symbol Device:R_Small -> can_controller-rescue:R_Small-Device
- R9: renamed from R3; footprint (none) -> Resistor_SMD:R_1206_3216Metric_Pad1.42x1.75mm_HandSolder; symbol Device:R_Small -> can_controller-rescue:R_Small-Device
- SW1: footprint (none) -> buttoni:SW_TL3305AF260QG; symbol Switch:SW_Push_Dual -> can_controller-rescue:SW_Push_Dual-Switch
- U2: symbol MCU_ST_STM32F1:STM32F105RCTx -> can_controller-rescue:STM32F105RCTx-MCU_ST_STM32F1
- U4, U5: symbol Interface_CAN_LIN:SN65HVD232 -> can_controller-rescue:SN65HVD232-Interface_CAN_LIN
- Y1: footprint (none) -> Crystal:Crystal_HC49-4H_Vertical; symbol Device:Crystal_Small -> can_controller-rescue:Crystal_Small-Device
Connections:
- net +3V3: now also C17.1, L2.2, R7.2
- net +5V: now also C4.1, L1.2, R2.2
- net 12V: now also C13.1, R1.1, R5.1, U1.5 (VIN), U3.5 (VIN)
- net GND: now also C13.2, C17.2, C4.2, D1.2 (A), D4.2 (A), R3.1, R8.1, U1.2 (GND), U3.2 (GND)
- new net: C2.1, U1.1 (BST)
- new net: R2.1, R3.2, U1.3 (FB)
- new net: R1.2, U1.4 (EN)
- new net: C2.2, D1.1 (K), L1.1, U1.6 (LX)
- new net: C14.1, U3.1 (BST)
- new net: R7.1, R8.2, U3.3 (FB)
- new net: R5.2, U3.4 (EN)
- new net: C14.2, D4.1 (K), L2.1, U3.6 (LX)
Other:
- moved on the sheet: C1
